Commit message: working example

File: yumi/yumi_description/urdf/yumi.urdf (robot description, URDF)
Before this commit: robot yumi, 23 links, 22 joints
Joints:
- joint yumi_robl_joint_3: child yumi_link_4_l -> yumi_link_3_l; limit lower=-2.155481626212997 upper=1.3962634015954636 effort=300 velocity=3.141592653589793 -> lower=-2.940879789610445 upper=2.940879789610445 effort=300 velocity=3.141592653589793; origin xyz=-0.04188 0.0 0.07873 rpy=1.5707963267948966 -1.5707963267948966 0.0 -> xyz=-0.03 0.17283 0.0 rpy=-1.5707963267948966 0.0 0.0; parent yumi_link_3_l -> yumi_link_2_l
- joint yumi_robl_joint_4: child yumi_link_5_l -> yumi_link_4_l; limit lower=-5.061454830783555 upper=5.061454830783555 effort=300 velocity=6.981317007977318 -> lower=-2.155481626212997 upper=1.3962634015954636 effort=300 velocity=3.141592653589793; origin xyz=0.0405 0.16461 0.0 rpy=-1.5707963267948966 0.0 0.0 -> xyz=-0.04188 0.0 0.07873 rpy=1.5707963267948966 -1.5707963267948966 0.0; parent yumi_link_4_l -> yumi_link_3_l
- joint yumi_robl_joint_5: child yumi_link_6_l -> yumi_link_5_l; limit lower=-1.53588974175501 upper=2.4085543677521746 effort=300 velocity=6.981317007977318 -> lower=-5.061454830783555 upper=5.061454830783555 effort=300 velocity=6.981317007977318; origin xyz=-0.027 0 0.10039 rpy=1.5707963267948966 0.0 0.0 -> xyz=0.0405 0.16461 0.0 rpy=-1.5707963267948966 0.0 0.0; parent yumi_link_5_l -> yumi_link_4_l
- joint yumi_robl_joint_6: child yumi_link_7_l -> yumi_link_6_l; limit lower=-3.9968039870670142 upper=3.9968039870670142 effort=300 velocity=6.981317007977318 -> lower=-1.53588974175501 upper=2.4085543677521746 effort=300 velocity=6.981317007977318; origin xyz=0.027 0.029 0.0 rpy=-1.5707963267948966 0.0 0.0 -> xyz=-0.027 0 0.10039 rpy=1.5707963267948966 0.0 0.0; parent yumi_link_6_l -> yumi_link_5_l
- joint yumi_robl_joint_7: child yumi_link_3_l -> yumi_link_7_l; limit lower=-2.940879789610445 upper=2.940879789610445 effort=300 velocity=3.141592653589793 -> lower=-3.9968039870670142 upper=3.9968039870670142 effort=300 velocity=6.981317007977318; origin xyz=-0.03 0.17283 0.0 rpy=-1.5707963267948966 0.0 0.0 -> xyz=0.027 0.029 0.0 rpy=-1.5707963267948966 0.0 0.0; parent yumi_link_2_l -> yumi_link_6_l
- joint yumi_robr_joint_3: child yumi_link_4_r -> yumi_link_3_r; limit lower=-2.155481626212997 upper=1.3962634015954636 effort=300 velocity=3.141592653589793 -> lower=-2.940879789610445 upper=2.940879789610445 effort=300 velocity=3.141592653589793; origin xyz=-0.04188 0.0 0.07873 rpy=1.5707963267948966 -1.5707963267948966 0.0 -> xyz=-0.03 0.17283 0.0 rpy=-1.5707963267948966 0.0 0.0; parent yumi_link_3_r -> yumi_link_2_r
- joint yumi_robr_joint_4: child yumi_link_5_r -> yumi_link_4_r; limit lower=-5.061454830783555 upper=5.061454830783555 effort=300 velocity=6.981317007977318 -> lower=-2.155481626212997 upper=1.3962634015954636 effort=300 velocity=3.141592653589793; origin xyz=0.0405 0.16461 0.0 rpy=-1.5707963267948966 0.0 0.0 -> xyz=-0.04188 0.0 0.07873 rpy=1.5707963267948966 -1.5707963267948966 0.0; parent yumi_link_4_r -> yumi_link_3_r
- joint yumi_robr_joint_5: child yumi_link_6_r -> yumi_link_5_r; limit lower=-1.53588974175501 upper=2.4085543677521746 effort=300 velocity=6.981317007977318 -> lower=-5.061454830783555 upper=5.061454830783555 effort=300 velocity=6.981317007977318; origin xyz=-0.027 0 0.10039 rpy=1.5707963267948966 0.0 0.0 -> xyz=0.0405 0.16461 0.0 rpy=-1.5707963267948966 0.0 0.0; parent yumi_link_5_r -> yumi_link_4_r
- joint yumi_robr_joint_6: child yumi_link_7_r -> yumi_link_6_r; limit lower=-3.9968039870670142 upper=3.9968039870670142 effort=300 velocity=6.981317007977318 -> lower=-1.53588974175501 upper=2.4085543677521746 effort=300 velocity=6.981317007977318; origin xyz=0.027 0.029 0.0 rpy=-1.5707963267948966 0.0 0.0 -> xyz=-0.027 0 0.10039 rpy=1.5707963267948966 0.0 0.0; parent yumi_link_6_r -> yumi_link_5_r
- joint yumi_robr_joint_7: child yumi_link_3_r -> yumi_link_7_r; limit lower=-2.940879789610445 upper=2.940879789610445 effort=300 velocity=3.141592653589793 -> lower=-3.9968039870670142 upper=3.9968039870670142 effort=300 velocity=6.981317007977318; origin xyz=-0.03 0.17283 0.0 rpy=-1.5707963267948966 0.0 0.0 -> xyz=0.027 0.029 0.0 rpy=-1.5707963267948966 0.0 0.0; parent yumi_link_2_r -> yumi_link_6_r

File: yumi/yumi_description/urdf/yumi.urdf.xacro (robot description, xacro)
@@ -11,7 +11,5 @@
   <!-- Import Gazebo plugins -->
   <xacro:include filename="$(find yumi_description)/urdf/Gazebo/gazebo.urdf.xacro"/>
-  <xacro:arg name="arms_interface" default="VelocityJointInterface"/>
-  <xacro:arg name="grippers_interface" default="EffortJointInterface"/>
-  <xacro:property name="yumi_parent" value="world" />
+  <!--yumi-->
   <link name="world"/>
   <joint name="world_joint" type="fixed">
@@ -20,14 +18,13 @@
     <origin xyz="0 0 0.1" rpy="0 0 0" />
   </joint>
-  <!--yumi-->
-  <xacro:yumi name="yumi" hardware_interface="hardware_interface/$(arg arms_interface)" parent="world" >
+  <xacro:yumi name="yumi" hardware_interface="hardware_interface/VelocityJointInterface" parent="world" >
     <origin xyz="0 0 0.1" rpy="0 0 0" />
   </xacro:yumi>
   <!--right gripper-->
-  <xacro:yumi_servo_gripper name="gripper_r" hardware_interface="hardware_interface/$(arg grippers_interface)" parent="yumi_link_7_r">
+  <xacro:yumi_servo_gripper name="gripper_r" hardware_interface="hardware_interface/EffortJointInterface" parent="yumi_link_7_r">
     <origin xyz="0 0 0.007" rpy="0 0 ${PI}" />
   </xacro:yumi_servo_gripper>
   <!--left gripper-->
-  <xacro:yumi_servo_gripper name="gripper_l" hardware_interface="hardware_interface/$(arg grippers_interface)" parent="yumi_link_7_l">
+  <xacro:yumi_servo_gripper name="gripper_l" hardware_interface="hardware_interface/EffortJointInterface" parent="yumi_link_7_l">
     <origin xyz="0 0 0.007" rpy="0 0 ${PI}" />
   </xacro:yumi_servo_gripper>

File: yumi/yumi_description/urdf/yumi.xacro (robot description, xacro)
@@ -99,14 +99,14 @@
       </collision>
     </link>
-  <!-- joint between link_2_r and link_3_r -->
-    <joint name="${name}_robr_joint_7" type="revolute">
-      <parent link="${name}_link_2_r"/>
-      <child link="${name}_link_3_r"/>
-      <origin xyz="-0.03 0.17283 0.0" rpy="${-PI / 2} 0.0 0.0"/>
-      <axis xyz="0 0 1"/>
-      <limit lower="${-168.5 * PI / 180}" upper="${168.5 * PI / 180}"
-              effort="${max_effort}" velocity="${180 * PI / 180}" />
-      <dynamics damping="${joint_damping}"/>
-    </joint>
+     <!-- joint between link_2_r and link_3_r -->
+      <joint name="${name}_robr_joint_3" type="revolute">
+        <parent link="${name}_link_2_r"/>
+        <child link="${name}_link_3_r"/>
+        <origin xyz="-0.03 0.17283 0.0" rpy="${-PI / 2} 0.0 0.0"/>
+        <axis xyz="0 0 1"/>
+        <limit lower="${-168.5 * PI / 180}" upper="${168.5 * PI / 180}"
+               effort="${max_effort}" velocity="${180 * PI / 180}" />
+        <dynamics damping="${joint_damping}"/>
+      </joint>
     <link name="${name}_link_3_r">
       <inertial>
@@ -131,5 +131,5 @@
     </link>
     <!-- joint between link_3_r and link_4_r -->
-    <joint name="${name}_robr_joint_3" type="revolute">
+    <joint name="${name}_robr_joint_4" type="revolute">
       <parent link="${name}_link_3_r"/>
       <child link="${name}_link_4_r"/>
@@ -162,5 +162,5 @@
     </link>
     <!-- joint between link_4_r and link_5_r -->
-    <joint name="${name}_robr_joint_4" type="revolute">
+    <joint name="${name}_robr_joint_5" type="revolute">
       <parent link="${name}_link_4_r"/>
       <child link="${name}_link_5_r"/>
@@ -193,5 +193,5 @@
     </link>
     <!-- joint between link_5_r and link_6_r -->
-    <joint name="${name}_robr_joint_5" type="revolute">
+    <joint name="${name}_robr_joint_6" type="revolute">
       <parent link="${name}_link_5_r"/>
       <child link="${name}_link_6_r"/>
@@ -224,5 +224,5 @@
     </link>
     <!-- joint between link_6_r and link_7_r -->
-    <joint name="${name}_robr_joint_6" type="revolute">
+    <joint name="${name}_robr_joint_7" type="revolute">
       <parent link="${name}_link_6_r"/>
       <child link="${name}_link_7_r"/>
@@ -318,5 +318,5 @@
     </link>
     <!-- joint between link_2_l and link_3_l -->
-    <joint name="${name}_robl_joint_7" type="revolute">
+    <joint name="${name}_robl_joint_3" type="revolute">
       <parent link="${name}_link_2_l"/>
       <child link="${name}_link_3_l"/>
@@ -349,5 +349,5 @@
     </link>
     <!-- joint between link_3_l and link_4_l -->
-    <joint name="${name}_robl_joint_3" type="revolute">
+    <joint name="${name}_robl_joint_4" type="revolute">
       <parent link="${name}_link_3_l"/>
       <child link="${name}_link_4_l"/>
@@ -380,5 +380,5 @@
     </link>
     <!-- joint between link_4_l and link_5_l -->
-    <joint name="${name}_robl_joint_4" type="revolute">
+    <joint name="${name}_robl_joint_5" type="revolute">
       <parent link="${name}_link_4_l"/>
       <child link="${name}_link_5_l"/>
@@ -411,5 +411,5 @@
     </link>
     <!-- joint between link_5_l and link_6_l -->
-    <joint name="${name}_robl_joint_5" type="revolute">
+    <joint name="${name}_robl_joint_6" type="revolute">
       <parent link="${name}_link_5_l"/>
       <child link="${name}_link_6_l"/>
@@ -442,5 +442,5 @@
     </link>
     <!-- joint between link_6_l and link_7_l -->
-    <joint name="${name}_robl_joint_6" type="revolute">
+    <joint name="${name}_robl_joint_7" type="revolute">
       <parent link="${name}_link_6_l"/>
       <child link="${name}_link_7_l"/>
